File: Controller_Version_1/Controller v1.1.kicad_pcb (KiCad board)
At the start: 2 copper layers, 74.5 x 52.1 mm, 98 parts, among them J1 B2B-PH-K (JST), J2 B4B-PH-K (JST), J3 B5B-PH-K (JST), J4 B3B-PH-K (JST), Q1 2N7002 (Changjiang Electronic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, Q2 SI2301CDS-T1-GE3 (Vishay Inte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, Q3 2N7002 (Changjiang Electronic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, Q4 DMG4407SSS-13 (Diodes Incorpo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, SW1 5.1mm switch, U1 Feather nRF52840 Express (Ada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, U2 LMV321 (Texas Instruments), U3 OPA197IDR (Texas Instruments), U4 DRV8313PWP (Texas Instruments), U5 LMV321 (Texas Instruments), U6 LMV321 (Texas Instruments), U7 LMV321 (Texas Instruments)

Commit message: [PCB] Version ready for order
Parts:
- renumbered scl to TP1, vsn to TP10, isn to TP11, nft to TP12, en1 to TP13, en2 to TP14, en3 to TP15, in1 to TP16, in2 to TP17, in3 to TP18, is2 to TP19, sda to TP2, is1 to TP20, is3 to TP21, ref to TP3, hp1 to TP4, ha1 to TP5, hp2 to TP6, ha2 to TP7, hp3 to TP8, ha3 to TP9
Connections:
- U4 pad 19: (no net) -> gnd
- U4 pad 21: (no net) -> gnd
Routing:
- net curr_amp[2].output: track 42.0 -> 43.1 mm, vias 1 -> 2
- net curr_amp[1].output: vias 2 -> 3
Other:
- board text added: "en1"
- board text added: "en2"
- board text added: "en3"
- board text added: "ha1"
- board text added: "ha2"
- board text added: "ha3"
- board text added: "hp1"
- board text added: "hp2"
- board text added: "hp3"
- board text added: "in1"
- board text added: "in2"
- board text added: "in3"
- board text added: "is1"
- board text added: "is2"
- board text added: "is3"
- board text added: "isn"
- board text added: "nft"
- board text added: "ref"
- board text added: "scl"
- board text added: "sda"
- board text added: "vsn"
